File: PCB/GD_test/GD_test.kicad_sch (KiCad schematic)
At the start: 14 parts, among them Q1 EPC2051, Q2 EPC2070, Q3 EPC2014C, U1 LMG1020YFF, U2 TLV3501

Commit message: gate driver board
Parts:
- removed C5: C_Small, symbol Device:C_Small
- removed Q1: EPC2051, symbol Simulation_SPICE:NMOS
- removed Q2: EPC2070, symbol Simulation_SPICE:NMOS
- removed Q3: EPC2014C, symbol Simulation_SPICE:NMOS
- removed R1: 50, Resistor_SMD:R_0603_1608Metric, symbol Device:R_Small_US
- removed R2: OPEN, Resistor_SMD:R_0603_1608Metric, symbol Device:R_Small_US
- removed R3: SHORT, Resistor_SMD:R_0603_1608Metric, symbol Device:R_Small_US
- removed U2: TLV3501, Package_TO_SOT_SMD:SOT-23-6, symbol MyKICAD:TLV3501
- added C10, C15, C16, C17, C7, C8, C9: C_Small, Resistor_SMD:R_0603_1608Metric_Pad0.98x0.95mm_HandSolder, symbol Device:C_Small
- added C12, C14: C_Small, Resistor_SMD:R_0402_1005Metric_Pad0.72x0.64mm_HandSolder, symbol Device:C_Small
- added J4 (x4): RF_IN, Connector_Coaxial:SMA_Amphenol_132134-10_Vertical, symbol Connector:Conn_Coaxial
- added J5, J6: Conn_01x01_Pin, Connector:Banana_Jack_1Pin, symbol Connector:Conn_01x01_Pin
- added Q1, Q2: EPC2051, EPCGaN:BGA-6_3x2_6.0x6.0mm, symbol Device:Q_NMOS_GSD
- added Q3: EPC2070, EPCGaN:BGA-6_3x2_6.0x6.0mm, symbol Device:Q_NMOS_GSD
- added Q5: EPC2014C, EPCGaN:EPC2014C, symbol Device:Q_NMOS_GSD
- added R1 (x4): 50, Resistor_SMD:R_0603_1608Metric, symbol Device:R_Small_US
- added R2 (x4): OPEN, Resistor_SMD:R_0603_1608Metric, symbol Device:R_Small_US
- added R3 (x4): SHORT, Resistor_SMD:R_0603_1608Metric, symbol Device:R_Small_US
- added U1 (x4): TLV3501, Package_TO_SOT_SMD:SOT-23-6, symbol MyKICAD:TLV3501
- added U11, U9: LMG1020YFF, GateDriver:BGA6N40P3X2_125X85X62N, symbol Driver_FET:LMG1020YFF
- added U3, U5, U6, U7: NC7WZ04, pcbparts:SOIC-6, symbol parts:NC7WZ04
- C1, C2, C3, C4: footprint (none) -> Resistor_SMD:R_0603_1608Metric_Pad0.98x0.95mm_HandSolder
- C6: footprint (none) -> Resistor_SMD:R_0402_1005Metric_Pad0.72x0.64mm_HandSolder
- U1: footprint Package_BGA:Texas_DSBGA-6_0.855x1.255mm_Layout2x3_P0.4mm_LevelB -> GateDriver:BGA6N40P3X2_125X85X62N
Connections:
- net +5V: now also C10.1, C12.1, C14.1, C15.1, C16.1, C17.1, C7.1, C8.1, C9.1, J5.1 (Pin_1), R2.1, R2.1, R2.1, R2.1, U1.4 (V+), U1.4 (V+), U1.4 (V+), U1.4 (V+), U11.A1 (V_{DD}), U3.5 (VCC), U5.5 (VCC), U6.5 (VCC), U7.5 (VCC), U9.A1 (V_{DD})
- net GND: now also U1.C2 (IN-), C10.2, C12.2, C14.2, C15.2, C16.2, C17.2, C7.2, C8.2, C9.2, J4.2 (Ext), J4.2 (Ext), J4.2 (Ext), J4.2 (Ext), J6.1 (Pin_1), Q1.2 (S), Q1.3 (D), Q1.4 (D), Q1.5 (D), Q1.6 (D), Q2.2 (S), Q2.3 (D), Q2.4 (D), Q2.5 (D), Q2.6 (D), Q3.2 (S), Q3.3 (D), Q3.4 (D), Q3.5 (D), Q3.6 (D), Q5.2 (S), Q5.3 (D), Q5.4 (S), Q5.5 (D), R1.1, R1.1, R1.1, R1.1, R3.2, R3.2, R3.2, R3.2, U1.2 (V-), U1.2 (V-), U1.2 (V-), U1.2 (V-), U1.6 (SHDN), U1.6 (SHDN), U1.6 (SHDN), U1.6 (SHDN), U11.B1 (GND), U11.C2 (IN-), U3.2 (GND), U3.3 (A2), U5.2 (GND), U5.4 (Y2), U6.2 (GND), U6.4 (Y2), U7.2 (GND), U7.4 (Y2), U9.B1 (GND), U9.C2 (IN-)
- net at U1.C1 (IN+): now also U1.5 (OUT)
- net at U1.A2 (OUTH), U1.B2 (OUTL): now also Q2.1 (G)
- new net: R2.2, R3.1, U1.1 (-IN) (x4)
- new net: Q1.1 (G), U5.6 (Y1), U6.6 (Y1), U7.6 (Y1)
- new net: Q5.1 (G), U9.A2 (OUTH), U9.B2 (OUTL)
- new net: U1.5 (OUT), U9.C1 (IN+)
- new net: Q3.1 (G), U11.A2 (OUTH), U11.B2 (OUTL)
- new net: U1.5 (OUT), U11.C1 (IN+)
- new net: U1.5 (OUT), U3.1 (A1)
- new net BUFF_OUT+: U3.6 (Y1), U5.1 (A1), U6.1 (A1), U7.1 (A1)
- new net BUFF_OUT-: U3.4 (Y2), U5.3 (A2), U6.3 (A2), U7.3 (A2)
- new net RF_IN_1: J4.1 (In), R1.2, U1.3 (+IN)
- new net RF_IN_2: J4.1 (In), R1.2, U1.3 (+IN)
- new net RF_IN_3: J4.1 (In), R1.2, U1.3 (+IN)
- new net RF_IN_4: J4.1 (In), R1.2, U1.3 (+IN)
Other:
- moved on the sheet: C1, C2, C3, C4, C6, U1

Commit message: gate driver gerbers and some extra changes
Parts:
- C1, C10, C15, C16, C2, C3, C4: footprint Resistor_SMD:R_0603_1608Metric_Pad0.98x0.95mm_HandSolder -> Capacitor_SMD:C_0603_1608Metric_Pad1.08x0.95mm_HandSolder
- C12, C14: footprint Resistor_SMD:R_0402_1005Metric_Pad0.72x0.64mm_HandSolder -> Capacitor_SMD:C_0603_1608Metric_Pad1.08x0.95mm_HandSolder
- C17, C7, C8, C9: footprint Resistor_SMD:R_0603_1608Metric_Pad0.98x0.95mm_HandSolder -> Capacitor_SMD:C_0402_1005Metric_Pad0.74x0.62mm_HandSolder
- C6: footprint Resistor_SMD:R_0402_1005Metric_Pad0.72x0.64mm_HandSolder -> Capacitor_SMD:C_0402_1005Metric_Pad0.74x0.62mm_HandSolder
Changed lines of the file:
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@@
       (effects (font (size 1.27 1.27)) (justify left))
     )
-    (property "Footprint" "Resistor_SMD:R_0402_1005Metric_Pad0.72x0.64mm_HandSolder" (at 142.24 72.39 0)
+    (property "Footprint" "Capacitor_SMD:C_0402_1005Metric_Pad0.74x0.62mm_HandSolder" (at 142.24 72.39 0)
       (effects (font (size 1.27 1.27)) hide)
     )
@@
       (effects (font (size 1.27 1.27)) (justify left))
     )
-    (property "Footprint" "Resistor_SMD:R_0603_1608Metric_Pad0.98x0.95mm_HandSolder" (at 119.38 62.23 0)
+    (property "Footprint" "Capacitor_SMD:C_0603_1608Metric_Pad1.08x0.95mm_HandSolder" (at 119.38 62.23 0)
       (effects (font (size 1.27 1.27)) hide)
     )
@@
       (effects (font (size 1.27 1.27)) (justify left))
     )
-    (property "Footprint" "Resistor_SMD:R_0603_1608Metric_Pad0.98x0.95mm_HandSolder" (at 109.22 62.23 0)
+    (property "Footprint" "Capacitor_SMD:C_0603_1608Metric_Pad1.08x0.95mm_HandSolder" (at 109.22 62.23 0)
       (effects (font (size 1.27 1.27)) hide)
     )
@@
       (effects (font (size 1.27 1.27)) (justify left))
     )
-    (property "Footprint" "Resistor_SMD:R_0603_1608Metric_Pad0.98x0.95mm_HandSolder" (at 156.21 146.05 0)
+    (property "Footprint" "Capacitor_SMD:C_0402_1005Metric_Pad0.74x0.62mm_HandSolder" (at 156.21 146.05 0)
       (effects (font (size 1.27 1.27)) hide)
     )
@@
       (effects (font (size 1.27 1.27)) (justify left))
     )
-    (property "Footprint" "Resistor_SMD:R_0603_1608Metric_Pad0.98x0.95mm_HandSolder" (at 114.3 62.23 0)
+    (property "Footprint" "Capacitor_SMD:C_0603_1608Metric_Pad1.08x0.95mm_HandSolder" (at 114.3 62.23 0)
       (effects (font (size 1.27 1.27)) hide)
     )
@@
       (effects (font (size 1.27 1.27)) (justify left))
     )
-    (property "Footprint" "Resistor_SMD:R_0603_1608Metric_Pad0.98x0.95mm_HandSolder" (at 228.6 118.11 0)
+    (property "Footprint" "Capacitor_SMD:C_0603_1608Metric_Pad1.08x0.95mm_HandSolder" (at 228.6 118.11 0)
       (effects (font (size 1.27 1.27)) hide)
     )
@@
       (effects (font (size 1.27 1.27)) (justify left))
     )
-    (property "Footprint" "Resistor_SMD:R_0402_1005Metric_Pad0.72x0.64mm_HandSolder" (at 262.89 71.12 0)
+    (property "Footprint" "Capacitor_SMD:C_0603_1608Metric_Pad1.08x0.95mm_HandSolder" (at 262.89 71.12 0)
       (effects (font (size 1.27 1.27)) hide)
     )
@@
       (effects (font (size 1.27 1.27)) (justify left))
     )
-    (property "Footprint" "Resistor_SMD:R_0603_1608Metric_Pad0.98x0.95mm_HandSolder" (at 64.77 123.19 0)
+    (property "Footprint" "Capacitor_SMD:C_0603_1608Metric_Pad1.08x0.95mm_HandSolder" (at 64.77 123.19 0)
       (effects (font (size 1.27 1.27)) hide)
     )
@@
       (effects (font (size 1.27 1.27)) (justify left))
     )
-    (property "Footprint" "Resistor_SMD:R_0402_1005Metric_Pad0.72x0.64mm_HandSolder" (at 262.89 110.49 0)
+    (property "Footprint" "Capacitor_SMD:C_0603_1608Metric_Pad1.08x0.95mm_HandSolder" (at 262.89 110.49 0)
       (effects (font (size 1.27 1.27)) hide)
     )
@@
       (effects (font (size 1.27 1.27)) (justify left))
     )
-    (property "Footprint" "Resistor_SMD:R_0603_1608Metric_Pad0.98x0.95mm_HandSolder" (at 104.14 62.23 0)
+    (property "Footprint" "Capacitor_SMD:C_0603_1608Metric_Pad1.08x0.95mm_HandSolder" (at 104.14 62.23 0)
       (effects (font (size 1.27 1.27)) hide)
     )
@@
       (effects (font (size 1.27 1.27)) (justify left))
     )
-    (property "Footprint" "Resistor_SMD:R_0603_1608Metric_Pad0.98x0.95mm_HandSolder" (at 156.21 130.81 0)
+    (property "Footprint" "Capacitor_SMD:C_0402_1005Metric_Pad0.74x0.62mm_HandSolder" (at 156.21 130.81 0)
       (effects (font (size 1.27 1.27)) hide)
     )
@@
       (effects (font (size 1.27 1.27)) (justify left))
     )
-    (property "Value" "C_Small" (at 111.76 120.65 0)
-      (effects (font (size 1.27 1.27)) (justify left))
-    )
-    (property "Footprint" "Resistor_SMD:R_0603_1608Metric_Pad0.98x0.95mm_HandSolder" (at 113.03 123.19 0)
+    (property "Value" "C_Small" (at 113.03 119.38 0)
+      (effects (font (size 1.27 1.27)) (justify left))
+    )
+    (property "Footprint" "Capacitor_SMD:C_0402_1005Metric_Pad0.74x0.62mm_HandSolder" (at 113.03 123.19 0)
       (effects (font (size 1.27 1.27)) hide)
     )
@@
       (effects (font (size 1.27 1.27)) (justify left))
     )
-    (property "Footprint" "Resistor_SMD:R_0603_1608Metric_Pad0.98x0.95mm_HandSolder" (at 156.21 115.57 0)
+    (property "Footprint" "Capacitor_SMD:C_0402_1005Metric_Pad0.74x0.62mm_HandSolder" (at 156.21 115.57 0)
       (effects (font (size 1.27 1.27)) hide)
     )
@@
       (effects (font (size 1.27 1.27)) (justify left))
     )
-    (property "Footprint" "Resistor_SMD:R_0603_1608Metric_Pad0.98x0.95mm_HandSolder" (at 227.33 78.74 0)
-      (effects (font (size 1.27 1.27)) hide)
-    )
+    (property "Footprint" "Capacitor_SMD:C_0603_1608Metric_Pad1.08x0.95mm_HandSolder" (at 227.33 78.74 0)
+      (effects (font (size 1.27 1.27)) hide)
+    )
