File: PCB/GD_test/_autosave-GD_test.kicad_sch (KiCad schematic)
At the start: 47 parts, among them J4 RF_IN, J5 Conn_01x01_Pin, J6 Conn_01x01_Pin, Q1 EPC2051, Q2 EPC2051, Q3 GS61004B-MR, Q5 EPC2014C, U1 LMG1020YFF, U1 TLV3501, U11 LMG1020YFF, U3 NC7WZ04, U5 NC7WZ04, U6 NC7WZ04, U7 NC7WZ04, U9 LMG1020YFF

Commit message: gate driver test board changes
Parts:
- Q3: footprint GS61004B-MR:TRANS_GS61004B-MR -> EPCGaN:TRANS_GS61004B-MR
Changed lines of the file:
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@@
       (effects (font (size 1.27 1.27)) (justify left))
     )
-    (property "Footprint" "GS61004B-MR:TRANS_GS61004B-MR" (at 292.1 120.65 0)
+    (property "Footprint" "EPCGaN:TRANS_GS61004B-MR" (at 292.1 120.65 0)
       (effects (font (size 1.27 1.27)) (justify bottom) hide)
     )
@@
       (effects (font (size 1.27 1.27)) (justify bottom) hide)
     )
+    (property "MPN" "" (at 292.1 120.65 0)
+      (effects (font (size 1.27 1.27)) hide)
+    )
     (pin "1")
