File: PCB/Full/phi2_50MHz_EPC2214/_autosave-phi2_50MHz_EPC2214.kicad_sch (KiCad schematic)
At the start: 60 parts, among them J2 RF_OUT, J4 RF_IN, J5 Conn_01x01_Pin, J6 Conn_01x01_Pin, Q1 EPC2214, U1 TLV3501, U1 TPS563203, U3 NC7WZ04, U5 NC7WZ04, U6 NC7WZ04, U7 NC7WZ04

Commit message: xcircuit stuff
Other:
- note added: "28 pF"
- note removed: "50 pF"
Changed lines of the file:
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@@
 		)
 	)
-	(text "50 pF"
+	(text "28 pF"
 		(exclude_from_sim no)
 		(at 242.316 115.062 0)
