File: PCB/Full/phi2_50MHz_EPC8010/_autosave-phi2_50MHz_EPC8010.kicad_pcb (KiCad board)
At the start: 2 copper layers, 89 x 89 mm, 63 parts, among them J1 RF_IN, J2 RF_OUT, J5 Conn_01x01_Pin, J6 Conn_01x01_Pin, Q1 EPC8010, U1 TPS563203, U4 TLV3501, U5 NC7WZ16, U6 NC7WZ16, U7 NC7WZ16

Commit message: added measurement data
Parts:
- turned J1 to 90 degrees
Changed lines of the file:
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@@
 	(footprint "Connector_Coaxial:SMA_Amphenol_132134-10_Vertical"
 		(layer "F.Cu")
-		(at 44.32 61.29)
+		(at 44.32 61.29 90)
 		(descr "https://www.amphenolrf.com/downloads/dl/file/id/4007/product/2974/132134_10_customer_drawing.pdf")
 		(tags "SMA SMD Female Jack Vertical")
 		(property "Reference" "J1"
-			(at 0 -4.75 0)
+			(at 0 -4.75 270)
 			(layer "F.SilkS")
 			(effects
@@
 		)
 		(property "Value" "RF_IN"
-			(at 0 4.75 0)
+			(at 0 4.75 270)
 			(layer "F.Fab")
 			(effects
@@
 		)
 		(property "Footprint" "Connector_Coaxial:SMA_Amphenol_132134-10_Vertical"
-			(at 0 0 0)
+			(at 0 0 90)
 			(unlocked yes)
 			(layer "F.Fab")
@@
 		)
 		(property "Datasheet" " ~"
-			(at 0 0 0)
+			(at 0 0 90)
 			(unlocked yes)
 			(layer "F.Fab")
@@
 		)
 		(property "Description" ""
-			(at 0 0 0)
+			(at 0 0 90)
 			(unlocked yes)
 			(layer "F.Fab")
@@
 		(attr smd)
 		(fp_line
-			(start -3.355 -0.94)
-			(end -3.355 0.94)
+			(start 3.355 -0.94)
+			(end 3.355 0.94)
 			(stroke
 				(width 0.12)
@@
 		)
 		(fp_line
-			(start 3.355 -0.94)
-			(end 3.355 0.94)
+			(start -3.355 -0.94)
+			(end -3.355 0.94)
 			(stroke
 				(width 0.12)
@@
 		(fp_line
 			(start -4.06 -4.06)
-			(end -4.06 4.06)
+			(end 4.06 -4.06)
 			(stroke
 				(width 0.05)
@@
 		(fp_line
 			(start -4.06 -4.06)
-			(end 4.06 -4.06)
+			(end -4.06 4.06)
 			(stroke
 				(width 0.05)
@@
 		(fp_line
 			(start 4.06 4.06)
-			(end -4.06 4.06)
+			(end 4.06 -4.06)
 			(stroke
 				(width 0.05)
@@
 		(fp_line
 			(start 4.06 4.06)
-			(end 4.06 -4.06)
+			(end -4.06 4.06)
 			(stroke
 				(width 0.05)
@@
 		)
 		(fp_line
-			(start -3.175 -3.175)
-			(end -3.175 3.175)
+			(start 3.175 -3.175)
+			(end 3.175 3.175)
 			(stroke
 				(width 0.1)
@@
 		)
 		(fp_line
-			(start -3.175 3.175)
-			(end 3.175 3.175)
+			(start -3.175 -3.175)
+			(end -3.175 3.175)
 			(stroke
 				(width 0.1)
@@
 		)
 		(fp_line
-			(start 3.175 -3.175)
+			(start -3.175 3.175)
 			(end 3.175 3.175)
 			(stroke
@@
 		)
 		(fp_text user "${REFERENCE}"
-			(at 0 0 0)
+			(at 0 0 270)
 			(layer "F.Fab")
 			(effects
@@
 		)
 		(pad "1" smd circle
-			(at 0 0 90)
+			(at 0 0 180)
 			(size 1.73 1.73)
 			(layers "F.Cu" "F.Paste" "F.Mask")
@@
 		)
 		(pad "2" smd custom
-			(at 0 -2.8 180)
+			(at 0 -2.8 270)
 			(size 7.11 1.51)
 			(layers "F.Cu" "F.Paste" "F.Mask")
@@
 		)
 		(pad "2" smd custom
-			(at 0 2.8)
+			(at 0 2.8 90)
 			(size 7.11 1.51)
 			(layers "F.Cu" "F.Paste" "F.Mask")
@@
 	)
 	(via
-		(at 42.545 64.26)
+		(at 47.29 63.065)
 		(size 1)
 		(drill 0.6)
@@
 	)
 	(via
-		(at 47.27 58.36)
+		(at 41.39 58.34)
 		(size 1)
 		(drill 0.6)
@@
 	)
 	(via
-		(at 47.27 63.185)
+		(at 46.215 58.34)
 		(size 1)
 		(drill 0.6)
@@
 	)
 	(via
-		(at 41.345 58.335)
+		(at 41.365 64.265)
 		(size 1)
 		(drill 0.6)
@@
 	)
 	(via
-		(at 41.32 64.26)
+		(at 47.29 64.29)
 		(size 1)
 		(drill 0.6)
@@
 	)
 	(via
-		(at 47.295 64.26)
+		(at 47.29 58.315)
 		(size 1)
 		(drill 0.6)
@@
 	)
 	(via
-		(at 41.32 63.11)
+		(at 46.14 64.29)
 		(size 1)
 		(drill 0.6)
@@
 	)
 	(via
-		(at 41.345 59.485)
+		(at 42.515 64.265)
 		(size 1)
 		(drill 0.6)
@@
 	)
 	(via
-		(at 42.52 58.335)
+		(at 41.365 63.09)
 		(size 1)
 		(drill 0.6)
@@
 	)
 	(via
-		(at 47.27 59.51)
+		(at 42.54 58.34)
 		(size 1)
 		(drill 0.6)
@@
 	)
 	(via
-		(at 46.095 64.26)
+		(at 47.29 59.515)
 		(size 1)
 		(drill 0.6)
@@
 	)
 	(via
-		(at 46.12 58.36)
+		(at 41.39 59.49)
 		(size 1)
 		(drill 0.6)
@@
 	)
 	(zone
-		(net 9)
-		(net_name "Net-(U1-SW)")
-		(layer "F.Cu")
-		(name "$teardrop_padvia$")
-		(hatch full 0.1)
-		(priority 30000)
-		(attr
-			(teardrop
-				(type padvia)
-			)
-		)
-		(connect_pads yes
-			(clearance 0)
-		)
-		(min_thickness 0.0254)
-		(filled_areas_thickness no)
-		(fill yes
-			(thermal_gap 0.5)
-			(thermal_bridge_width 0.5)
-			(island_removal_mode 1)
-			(island_area_min 10)
-		)
-		(polygon
-			(pts
-				(xy 26.57 41.69) (xy 26.87 41.69) (xy 26.89 41.435) (xy 26.72 41.169) (xy 26.55 41.435)
-			)
-		)
-	)
-	(zone
 		(net 2)
 		(net_name "+12V")
@@
 			)
 		)
+	)
+	(zone
+		(net 9)
+		(net_name "Net-(U1-SW)")
+		(layer "F.Cu")
+		(name "$teardrop_padvia$")
+		(hatch full 0.1)
+		(priority 30000)
+		(attr
+			(teardrop
+				(type padvia)
+			)
+		)
+		(connect_pads yes
+			(clearance 0)
+		)
+		(min_thickness 0.0254)
+		(filled_areas_thickness no)
+		(fill yes
+			(thermal_gap 0.5)
+			(thermal_bridge_width 0.5)
+			(island_removal_mode 1)
+			(island_area_min 10)
+		)
+		(polygon
+			(pts
+				(xy 26.57 41.69) (xy 26.87 41.69) (xy 26.89 41.435) (xy 26.72 41.169) (xy 26.55 41.435)
+			)
+		)
